File: LighthouseCircuit/ExenMiniMotorShield/ExenMiniMotorShield.sch (EAGLE design)
At the start: 13 parts, among them J3 SM02B-SRSS, Q1 DMP2035U

Commit message: Moved to separate PID configuration for each wheel. Since the left wheel is offset toward the rear and the right wheel is offset toward the front, the left wheel needs to be less aggressive or the Zippy will turn more quickly to the right and will tilt the robot and pull the right wheel off the ground, preventing contact with the floor. On the other hand, the right wheel needs to be more aggressive or turns to the left will be slower than turns to the right.
Parts:
- removed +5: (no value), SparkFun-Connectors:CONN_01PTH_NO_SILK_YES_STOP
- added A1, A2, A3, A4, D0, D1, MA01, MA02, MB01, MBO2, SCL, SDA, VIN: (no value), SparkFun-Connectors:CONN_01PTH_NO_SILK_YES_STOP
- added CB: 10μF, SparkFun-Capacitors:4.7PF-0603-50V-5%
- added MOC: A3901SEJTR-T, ZippyComponentLibrary:A3901SEJTR-T
- J3: value SM02B-SRSS -> BATTERY
Connections:
- removed net N$5: BC.VDD, Q1.S
- new net IO1: A1.1, MOC.IN4
- new net IO2: A2.1, MOC.IN3
- new net IO3: A3.1, MOC.IN2
- new net IO4: A4.1, MOC.IN1
- new net MA01: MBO2.1, MOC.OUT3
- new net MA02: MB01.1, MOC.OUT4
- new net MB01: MA02.1, MOC.OUT1
- new net MB02: MA01.1, MOC.OUT2
- new net VDD: BC.VDD, DBI.ANODE, Q1.S
- net GND: now also CB.1, MOC.EPAD, MOC.GND
- net VBAT: now also CB.2, MOC.VBB, Q1.G
- net VIN: now also VIN.1; no longer +5.1, DBI.ANODE, Q1.G
