File: LighthouseCircuit/ExenMiniShield/ExenMiniShield.sch (EAGLE design)
At the start: 30 parts

Commit message: Significantly stabilized the acceleration from full stop by slowing down the maximum speed. There is a physical limitation preventing them from accelerating any faster from full stop. Now that their wheels are offset, right turns cause the right wheel to lift up from the ground, creating error differences that the PID controllers are not setup to accommodate.
Parts:
- added J3: SM02B-SRSS, tinycircuits:AS-ITM-00231
Connections:
- net D1IN: now also OAG1.IN-; no longer OAG4.IN-
- net D1OA2P: now also OAG4.IN-; no longer OAG3.IN-
- net D1OAOUT1: now also OAG1.OUT; no longer OAG4.OUT
- net D2IN: now also OAG2.IN-; no longer OAG1.IN-
- net D2OA1OUT: now also OAG2.OUT; no longer OAG1.OUT
- net D2OA2N: now also OAG3.IN+; no longer OAG2.IN+
- net D2OA2P: now also OAG3.IN-; no longer OAG2.IN-
- net GND: now also J3.2
- net IO3: now also OAG3.OUT; no longer OAG2.OUT
- net IO7: now also OAG4.OUT; no longer OAG3.OUT
- net LVCC: now also OAG2.IN+; no longer OAG4.IN+
- net N$11: now also OAG4.IN+; no longer OAG3.IN+
- net VBAT: now also J3.1
Other:
- moved on the sheet: OAG1, OAG2, OAG3, OAG4
Changed lines of the file:
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@@
 <part name="+5V" library="SparkFun-Connectors" deviceset="CONN_01" device="PTH_NO_SILK_YES_STOP"/>
 <part name="GND" library="ZippyComponentLibrary" deviceset="SINGLE-THROUGH-HOLE" device=""/>
+<part name="J3" library="tinycircuits" deviceset="AS-ITM-00231" device="" value="SM02B-SRSS"/>
 </parts>
 <sheets>
@@
 <instance part="R3B" gate="G$1" x="261.62" y="-20.32" rot="MR270"/>
 <instance part="R4B" gate="G$1" x="274.32" y="-12.7"/>
-<instance part="OA" gate="G4" x="200.66" y="7.62"/>
-<instance part="OA" gate="G1" x="200.66" y="88.9"/>
-<instance part="OA" gate="G2" x="274.32" y="86.36"/>
-<instance part="OA" gate="G3" x="274.32" y="5.08"/>
+<instance part="OA" gate="G1" x="200.66" y="7.62"/>
+<instance part="OA" gate="G2" x="200.66" y="88.9"/>
+<instance part="OA" gate="G3" x="274.32" y="86.36"/>
+<instance part="OA" gate="G4" x="274.32" y="5.08"/>
 <instance part="OA" gate="PWR" x="152.4" y="53.34" rot="R90"/>
 <instance part="IO7" gate="G$1" x="304.8" y="5.08" smashed="yes" rot="R180">
@@
 <wire x1="190.5" y1="86.36" x2="187.96" y2="86.36" width="0.1524" layer="91"/>
 <label x="185.42" y="78.74" size="1.778" layer="95"/>
+<pinref part="OA" gate="G2" pin="IN+"/>
+<wire x1="187.96" y1="86.36" x2="187.96" y2="81.28" width="0.1524" layer="91"/>
+</segment>
+<segment>
 <pinref part="OA" gate="G1" pin="IN+"/>
-<wire x1="187.96" y1="86.36" x2="187.96" y2="81.28" width="0.1524" layer="91"/>
-</segment>
-<segment>
-<pinref part="OA" gate="G4" pin="IN+"/>
 <wire x1="190.5" y1="5.08" x2="187.96" y2="5.08" width="0.1524" layer="91"/>
 <wire x1="187.96" y1="5.08" x2="187.96" y2="0" width="0.1524" layer="91"/>
@@
 <wire x1="241.3" y1="88.9" x2="264.16" y2="88.9" width="0.1524" layer="91"/>
 <junction x="241.3" y="88.9"/>
-<pinref part="OA" gate="G2" pin="IN-"/>
+<pinref part="OA" gate="G3" pin="IN-"/>
 </segment>
 </net>
@@
 <junction x="261.62" y="71.12"/>
 <wire x1="264.16" y1="83.82" x2="261.62" y2="83.82" width="0.1524" layer="91"/>
-<pinref part="OA" gate="G2" pin="IN+"/>
+<pinref part="OA" gate="G3" pin="IN+"/>
 </segment>
 </net>
@@
 <junction x="215.9" y="88.9"/>
 <junction x="215.9" y="88.9"/>
-<pinref part="OA" gate="G1" pin="OUT"/>
+<pinref part="OA" gate="G2" pin="OUT"/>
 </segment>
 </net>
@@
 <wire x1="215.9" y1="7.62" x2="215.9" y2="33.02" width="0.1524" layer="91"/>
 <wire x1="215.9" y1="33.02" x2="210.82" y2="33.02" width="0.1524" layer="91"/>
-<pinref part="OA" gate="G4" pin="OUT"/>
+<pinref part="OA" gate="G1" pin="OUT"/>
 <pinref part="C2B" gate="G$1" pin="1"/>
 <wire x1="226.06" y1="7.62" x2="215.9" y2="7.62" width="0.1524" layer="91"/>
@@
 <wire x1="241.3" y1="7.62" x2="241.3" y2="2.54" width="0.1524" layer="91"/>
 <wire x1="241.3" y1="7.62" x2="264.16" y2="7.62" width="0.1524" layer="91"/>
-<pinref part="OA" gate="G3" pin="IN-"/>
+<pinref part="OA" gate="G4" pin="IN-"/>
 <pinref part="C2B" gate="G$1" pin="2"/>
 <wire x1="236.22" y1="7.62" x2="241.3" y2="7.62" width="0.1524" layer="91"/>
@@
 <wire x1="187.96" y1="111.76" x2="190.5" y2="111.76" width="0.1524" layer="91"/>
 <junction x="187.96" y="91.44"/>
-<pinref part="OA" gate="G1" pin="IN-"/>
+<pinref part="OA" gate="G2" pin="IN-"/>
 <pinref part="D1" gate="G$1" pin="CATHODE"/>
 <junction x="179.07" y="91.44"/>
@@
 <wire x1="187.96" y1="33.02" x2="190.5" y2="33.02" width="0.1524" layer="91"/>
 <junction x="187.96" y="10.16"/>
-<pinref part="OA" gate="G4" pin="IN-"/>
+<pinref part="OA" gate="G1" pin="IN-"/>
 <pinref part="C1B" gate="G$1" pin="1"/>
 <wire x1="195.58" y1="38.1" x2="190.5" y2="33.02" width="0.1524" layer="91"/>
@@
 <net name="N$11" class="0">
 <segment>
-<pinref part="OA" gate="G3" pin="IN+"/>
+<pinref part="OA" gate="G4" pin="IN+"/>
 <wire x1="261.62" y1="2.54" x2="264.16" y2="2.54" width="0.1524" layer="91"/>
 <pinref part="R4B" gate="G$1" pin="1"/>
@@
 <pinref part="R4A" gate="G$1" pin="2"/>
 <wire x1="279.4" y1="71.12" x2="289.56" y2="71.12" width="0.1524" layer="91"/>
-<pinref part="OA" gate="G2" pin="OUT"/>
+<pinref part="OA" gate="G3" pin="OUT"/>
 <wire x1="287.02" y1="86.36" x2="289.56" y2="86.36" width="0.1524" layer="91"/>
 <wire x1="289.56" y1="86.36" x2="297.18" y2="86.36" width="0.1524" layer="91"/>
@@
 <net name="IO7" class="0">
 <segment>
-<pinref part="OA" gate="G3" pin="OUT"/>
+<pinref part="OA" gate="G4" pin="OUT"/>
 <wire x1="287.02" y1="5.08" x2="289.56" y2="5.08" width="0.1524" layer="91"/>
 <pinref part="R4B" gate="G$1" pin="2"/>
@@
 <attribute name="VALUE" x="-37.846" y="22.86" size="1.778" layer="96" font="vector" rot="R270"/>
 </instance>
+<instance part="J3" gate="G$1" x="86.36" y="5.08" rot="MR180"/>
 </instances>
 <busses>
@@
 <label x="40.64" y="-10.16" size="1.778" layer="95"/>
 <pinref part="U$1" gate="BC" pin="VSS"/>
+</segment>
+<segment>
+<pinref part="J3" gate="G$1" pin="2"/>
+<wire x1="76.2" y1="5.08" x2="71.12" y2="5.08" width="0.1524" layer="91"/>
 </segment>
 </net>
@@
 <pinref part="U$1" gate="BC" pin="VBAT"/>
 </segment>
-</net>
+<segment>
+<pinref part="J3" gate="G$1" pin="1"/>
+<wire x1="76.2" y1="2.54" x2="71.12" y2="2.54" width="0.1524" layer="91"/>
+</segment>
+</net>

Commit message: Reached a point where auto-drive mode is consistent and reliable.
Parts:
- removed +5V, IO3, IO7: (no value), SparkFun-Connectors:CONN_01PTH_NO_SILK_YES_STOP
- removed C1BAT: 10uF, ZippyComponentLibrary:CAPACITOR
- removed C2BAT: 4.7uF, ZippyComponentLibrary:CAPACITOR
- removed D2: PHOTODIODEBPW, ZippyComponentLibrary:PHOTODIODEBPW
- removed U$1: BATTERYCHARGER, ZippyComponentLibrary:BATTERYCHARGER
- added A1, A2, A3, A4, D0, MA01, MA02, MB01, MBO2, VIN: (no value), SparkFun-Connectors:CONN_01PTH_NO_SILK_YES_STOP
- added BC: BATTERYCHARGER, ZippyComponentLibrary:BATTERYCHARGER
- added C1: 10uF, ZippyComponentLibrary:CAPACITOR
- added C2: 4.7uF, ZippyComponentLibrary:CAPACITOR
- added CB: 10μF, SparkFun-Capacitors:4.7PF-0603-50V-5%
- added D3: MBR120, tinycircuits:AS-ITM-00111
- added DI0, DI1: PHOTODIODEBPW, ZippyComponentLibrary:PHOTODIODEBPW
- added MOC: A3901SEJTR-T, ZippyComponentLibrary:A3901SEJTR-T
- added Q1: DMP2035U, tinycircuits:AS-ITM-00024
- D1: value PHOTODIODEBPW -> (none); device ZippyComponentLibrary:PHOTODIODEBPW -> SparkFun-Connectors:CONN_01PTH_NO_SILK_YES_STOP
- GND: value SINGLE-THROUGH-HOLE -> (none); device ZippyComponentLibrary:SINGLE-THROUGH-HOLE -> SparkFun-Connectors:CONN_01PTH_NO_SILK_YES_STOP
- J3: value SM02B-SRSS -> BATTERY
- OA: value TLV2464IDM -> TLV2464IPW; device ZippyComponentLibrary:TLV2464IDM -> ZippyComponentLibrary:TLV2464IPW
Connections:
- removed net +5V: +5V.1, C1BAT.2, DBI.ANODE, U$1.VDD
- removed net IO3: IO3.1, OAG3.OUT, R4A.2
- removed net IO7: IO7.1, OAG4.OUT, R4B.2
- new net D0: D0.1, OAG2.OUT, R4A.2
- new net D1: D1.1, OAG3.OUT, R4B.2
- new net MA01: MBO2.1, MOC.OUT3
- new net MA02: MB01.1, MOC.OUT4
- new net MB01: MA02.1, MOC.OUT1
- new net MB02: MA01.1, MOC.OUT2
- new net N$4: A1.1, MOC.IN4
- new net N$5: A2.1, MOC.IN3
- new net N$6: A4.1, MOC.IN1
- new net N$7: A3.1, MOC.IN2
- new net VDD: BC.VDD, DBI.ANODE, Q1.S
- new net VIN: C1.2, D3.C, Q1.D, VIN.1
- net D1IN: now also DI1.CATHODE, OAG4.IN-; no longer D2.CATHODE, OAG1.IN-
- net D1OA2P: now also OAG3.IN-; no longer OAG4.IN-
- net D1OAOUT1: now also OAG4.OUT; no longer OAG1.OUT
- net D2IN: now also DI0.CATHODE, OAG1.IN-; no longer D1.CATHODE, OAG2.IN-
- net D2OA1OUT: now also OAG1.OUT; no longer OAG2.OUT
- net D2OA2N: now also OAG2.IN+; no longer OAG3.IN+
- net D2OA2P: now also OAG2.IN-; no longer OAG3.IN-
- net GND: now also BC.VSS, C1.1, C2.1, CB.1, MOC.EPAD, MOC.GND; no longer C1BAT.1, C2BAT.1, U$1.VSS
- net LVCC: now also DI0.ANODE, DI1.ANODE, OAG4.IN+; no longer D1.ANODE, D2.ANODE, OAG2.IN+
- net N$11: now also OAG3.IN+; no longer OAG4.IN+
- net N$2: now also BC.STAT; no longer U$1.STAT
- net N$3: now also BC.PROG; no longer U$1.PROG
- net VBAT: now also BC.VBAT, C2.2, CB.2, D3.A, MOC.VBB, Q1.G; no longer C2BAT.2, U$1.VBAT
