File: LighthouseCircuit/Horizontally_Mounted_Lighthouse.brd (EAGLE design)
At the start: 25.4 x 11.4 mm, 23 parts

Commit message: Significantly stabilized the position calculation and the new driving model with independent PIDs for each wheel.
Parts:
- OA: value TLV2464IDM -> TLV2464IPW; device ZippyComponentLibrary:D14-M -> ZippyComponentLibrary:PW14
- moved R2B 17.1 mm to (1.91, 8.89), turned to 0 degrees
- moved C1B 10.2 mm to (17.1, 9.53), turned to 180 degrees
- moved R4B 8.47 mm to (9.53, 9.53), turned to 0 degrees
- moved R1A 4.49 mm to (13.3, 1.91), turned to 0 degrees
- moved R1B 4.49 mm to (13.3, 9.53), turned to 180 degrees
- moved C2B 3.70 mm to (1.91, 6.99), turned to 180 degrees
- moved R3B 3.17 mm to (5.71, 9.53), turned to 180 degrees
- moved C1A 2.62 mm to (9.53, 1.91), turned to 0 degrees
- moved R2A 2.01 mm to (17.1, 1.91), turned to 0 degrees
- moved R4A 1.42 mm to (1.91, 5.08), turned to 0 degrees
- moved R3A 1.42 mm to (1.91, 3.17), turned to 0 degrees
- moved C2A 0.90 mm to (5.71, 1.91), turned to 0 degrees
- moved OA 0.63 mm to (14.0, 5.71)
- moved CO 0.63 mm to (20.3, 2.54), turned to 270 degrees
- moved RI 0.63 mm to (20.3, 8.89), turned to 90 degrees
Routing:
- net LVCC: track 62.9 -> 0.00 mm, vias 2 -> 0
- net D2IN: track 25.7 -> 0.00 mm, vias 1 -> 0
- net D1IN: track 19.5 -> 0.00 mm, vias 1 -> 0
- net IO7: track 16.6 -> 0.00 mm, vias 1 -> 0
- net IO3: track 16.2 -> 0.00 mm, vias 1 -> 0
- net D1OA2P: track 15.7 -> 0.00 mm
- net D2OA2P: track 14.7 -> 0.00 mm
- net VCC: track 14.3 -> 0.00 mm, vias 1 -> 0
- net GND: track 12.9 -> 0.00 mm
- net D1OAOUT1: track 11.8 -> 0.00 mm
- net D2OA1OUT: track 11.7 -> 0.00 mm
- net N$11: track 11.4 -> 0.00 mm
- net D2OA2N: track 11.2 -> 0.00 mm
Other:
- board size 25.4 x 11.4 mm -> 25.4 x 10.2 mm
