File: LighthouseCircuit/Horizontally_Mounted_Lighthouse.sch (EAGLE design)
At the start: 23 parts

Commit message: Significantly stabilized the position calculation and the new driving model with independent PIDs for each wheel.
Parts:
- OA: value TLV2464IDM -> TLV2464IPW; device ZippyComponentLibrary:TLV2464IDM -> ZippyComponentLibrary:TLV2464IPW
Changed lines of the file:
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@@
 <?xml version="1.0" encoding="utf-8"?>
 <!DOCTYPE eagle SYSTEM "eagle.dtd">
-<eagle version="8.6.3">
+<eagle version="9.1.0">
 <drawing>
 <settings>
@@
 <part name="R3B" library="ZippyComponentLibrary" deviceset="RESISTOR" device="" value="1k"/>
 <part name="R4B" library="ZippyComponentLibrary" deviceset="RESISTOR" device="" value="100k"/>
-<part name="OA" library="ZippyComponentLibrary" deviceset="TLV2464ID" device="M" value="TLV2464IDM"/>
+<part name="OA" library="ZippyComponentLibrary" deviceset="TLV2464" device="IPW" value="TLV2464IPW"/>
 <part name="IO7" library="SparkFun-Connectors" deviceset="CONN_01" device="PTH_NO_SILK_YES_STOP"/>
 <part name="IO3" library="SparkFun-Connectors" deviceset="CONN_01" device="PTH_NO_SILK_YES_STOP"/>
